File: counter-mega8.brd (EAGLE design)
At the start: 25 parts, among them IC1 MEGA8-P

Commit message: initial commit
Routing:
- net GND: track 0.79 -> 329.2 mm
- net N$3: track 0.00 -> 9.00 mm, vias 0 -> 2
- removed copper zone on layer 16, net GND
Changed lines of the file:
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@@
 <contactref element="OK1" pad="4"/>
 <contactref element="JP1" pad="1"/>
+<wire x1="0" y1="0" x2="54.5" y2="0" width="1.6764" layer="16"/>
+<wire x1="54.5" y1="0" x2="54.5" y2="46" width="1.6764" layer="16"/>
+<wire x1="54.5" y1="46" x2="54.5" y2="54.5" width="1.6764" layer="16"/>
+<wire x1="54.5" y1="54.5" x2="50.5" y2="54.5" width="1.6764" layer="16"/>
+<wire x1="50.5" y1="54.5" x2="0" y2="54.5" width="1.6764" layer="16"/>
+<wire x1="0" y1="54.5" x2="0" y2="43" width="1.6764" layer="16"/>
+<wire x1="0" y1="43" x2="0" y2="36.5" width="1.6764" layer="16"/>
+<wire x1="0" y1="36.5" x2="0" y2="23" width="1.6764" layer="16"/>
+<wire x1="0" y1="23" x2="0" y2="0" width="1.6764" layer="16"/>
+<wire x1="50.69" y1="51.27" x2="50.5" y2="51.27" width="0.4064" layer="16"/>
+<wire x1="50.5" y1="51.27" x2="50.5" y2="54.5" width="0.4064" layer="16"/>
+<wire x1="33.91" y1="46.03" x2="54.5" y2="46.03" width="0.4064" layer="16"/>
+<wire x1="54.5" y1="46.03" x2="54.5" y2="46" width="0.4064" layer="16"/>
+<wire x1="8.96" y1="43.19" x2="0" y2="43.19" width="0.4064" layer="16"/>
+<wire x1="0" y1="43.19" x2="0" y2="43" width="0.4064" layer="16"/>
+<wire x1="0" y1="23" x2="2" y2="23" width="0.4064" layer="16"/>
+<wire x1="23.63" y1="20.32" x2="23.5" y2="20.32" width="0.4064" layer="16"/>
+<wire x1="23.5" y1="20.32" x2="23.5" y2="18" width="0.4064" layer="16"/>
+<wire x1="23.5" y1="18" x2="10.93" y2="18" width="0.4064" layer="16"/>
+<wire x1="10.93" y1="18" x2="10.93" y2="20.32" width="0.4064" layer="16"/>
+<wire x1="18.55" y1="38.64" x2="18.5" y2="38.64" width="0.4064" layer="16"/>
+<wire x1="18.5" y1="38.64" x2="18.5" y2="36.5" width="0.4064" layer="16"/>
+<wire x1="18.5" y1="36.5" x2="0" y2="36.5" width="0.4064" layer="16"/>
 <wire x1="21.47" y1="43.47" x2="21.5" y2="43.47" width="0.4064" layer="16"/>
+<wire x1="22.4" y1="36.5" x2="24.26" y2="36.5" width="0.4064" layer="16"/>
+<wire x1="24.26" y1="36.5" x2="24.26" y2="34.58" width="0.4064" layer="16"/>
+<wire x1="22.4" y1="36.5" x2="22.4" y2="43.1" width="0.4064" layer="16"/>
 <wire x1="24.26" y1="34.58" x2="23.5" y2="34.58" width="0.4064" layer="16"/>
-<polygon width="0.4064" layer="16" isolate="0.4064">
-<vertex x="0" y="0"/>
-<vertex x="55" y="0"/>
-<vertex x="55" y="55"/>
-<vertex x="0" y="55"/>
-</polygon>
-<wire x1="10.93" y1="5.08" x2="10.93" y2="20.32" width="0" layer="19" extent="1-1"/>
+<wire x1="23.5" y1="34.58" x2="23.5" y2="33" width="0.4064" layer="16"/>
+<wire x1="23.5" y1="33" x2="21.09" y2="33" width="0.4064" layer="16"/>
+<wire x1="21.09" y1="33" x2="21.09" y2="31.02" width="0.4064" layer="16"/>
+<wire x1="10.93" y1="20.32" x2="11" y2="20.32" width="0.4064" layer="16"/>
+<wire x1="11" y1="20.32" x2="11" y2="25" width="0.4064" layer="16"/>
+<wire x1="11" y1="25" x2="21.09" y2="25" width="0.4064" layer="16"/>
+<wire x1="21.09" y1="25" x2="21.09" y2="31.02" width="0.4064" layer="16"/>
+<wire x1="22.4" y1="43.1" x2="21.5" y2="43.47" width="0" layer="19" extent="16-16"/>
+<wire x1="18.5" y1="36.5" x2="22.4" y2="36.5" width="0" layer="19" extent="16-16"/>
+<wire x1="10.93" y1="5.08" x2="0" y2="0" width="0" layer="19" extent="16-16"/>
 <wire x1="23.63" y1="5.08" x2="10.93" y2="5.08" width="0" layer="19" extent="1-1"/>
 </signal>
@@
 </signal>
 <signal name="N$3">
+<via x="2" y="23" extent="1-16" drill="0.6" shape="square"/>
+<via x="11" y="23" extent="1-16" drill="0.6" shape="square"/>
+<wire x1="2" y1="23" x2="11" y2="23" width="0.4064" layer="1"/>
 </signal>
 </signals>
